File: CMRI-Bus-Interface-L_array.brd (EAGLE design)
At the start: 109.9 x 112.3 mm, 49 parts, among them CON1X11 0.100, CON1X21 0.100, CON2X11 0.100, CON2X21 0.100, M1X11 MOUNTINGHOLE, M1X21 MOUNTINGHOLE, M2X11 MOUNTINGHOLE, M2X21 MOUNTINGHOLE, M3X11 MOUNTINGHOLE, M3X21 MOUNTINGHOLE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

Commit message: added values for connectors
Parts:
- FID-LR, FID-UL: value (none) -> FID
- J1X11, J1X21: value (none) -> 0.100
- U2X1: value (none) -> 10x10
Changed lines of the file:
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@@
 <element name="CON2X11" library="SPCoast" package="1X05_LOCK" value="0.100" x="22.225" y="50.165" rot="R90"/>
 <element name="D1X11" library="SPCoast" package="SOT23" value="BAV199" x="15.24" y="19.685" rot="R90"/>
-<element name="J1X11" library="SPCoast" package="J3-254" value="" x="36.195" y="47.625" rot="R90"/>
+<element name="J1X11" library="SPCoast" package="J3-254" value="0.100" x="36.195" y="47.625" rot="R90"/>
 <element name="M1X11" library="SPCoast" package="MOUNTINGHOLE" value="MOUNTINGHOLE" x="7.62" y="15.875"/>
 <element name="M2X11" library="SPCoast" package="MOUNTINGHOLE" value="MOUNTINGHOLE" x="7.62" y="83.185"/>
@@
 <element name="CON2X21" library="SPCoast" package="1X05_LOCK" value="0.100" x="72.225" y="50.165" rot="R90"/>
 <element name="D1X21" library="SPCoast" package="SOT23" value="BAV199" x="65.24" y="19.685" rot="R90"/>
-<element name="J1X21" library="SPCoast" package="J3-254" value="" x="86.195" y="47.625" rot="R90"/>
+<element name="J1X21" library="SPCoast" package="J3-254" value="0.100" x="86.195" y="47.625" rot="R90"/>
 <element name="M1X21" library="SPCoast" package="MOUNTINGHOLE" value="MOUNTINGHOLE" x="57.62" y="15.875"/>
 <element name="M2X21" library="SPCoast" package="MOUNTINGHOLE" value="MOUNTINGHOLE" x="57.62" y="83.185"/>
@@
 <element name="U1X21" library="SPCoast" package="SO14" value="MAX3465CSD" x="63.97" y="29.845" rot="R90"/>
 <element name="U2X21" library="SPCoast" package="SO08" value="NE555" x="72.86" y="19.685"/>
-<element name="U2X1" library="SPCoast" package="BOARD-10X8X2-TEMPLATE" value="" x="0" y="0"/>
-<element name="FID-UL" library="SPCoast" package="FIDUCIAL_1MM" value="" x="6.35" y="92.075"/>
-<element name="FID-LR" library="SPCoast" package="FIDUCIAL_1MM" value="" x="93.98" y="7.62"/>
+<element name="U2X1" library="SPCoast" package="BOARD-10X8X2-TEMPLATE" value="10x10" x="0" y="0"/>
+<element name="FID-UL" library="SPCoast" package="FIDUCIAL_1MM" value="FID" x="6.35" y="92.075"/>
+<element name="FID-LR" library="SPCoast" package="FIDUCIAL_1MM" value="FID" x="93.98" y="7.62"/>
 </elements>
 <signals>
