File: CMRI-Bus-Interface-L_array.brd (EAGLE design)
At the start: 109.9 x 112.3 mm, 49 parts, among them CON1X11 0.100, CON1X21 0.100, CON2X11 0.100, CON2X21 0.100, J1X11 0.100, J1X21 0.100, M1X11 MOUNTINGHOLE, M1X21 MOUNTINGHOLE, M2X11 MOUNTINGHOLE, M2X21 MOUNTINGHOLE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

Commit message: normalized values
Parts:
- FID-LR, FID-UL: value FID -> FIDUCIAL
- U2X1: value 10x10 -> BOARD
Changed lines of the file:
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@@
 <element name="U1X21" library="SPCoast" package="SO14" value="MAX3465CSD" x="63.97" y="29.845" rot="R90"/>
 <element name="U2X21" library="SPCoast" package="SO08" value="NE555" x="72.86" y="19.685"/>
-<element name="U2X1" library="SPCoast" package="BOARD-10X8X2-TEMPLATE" value="10x10" x="0" y="0"/>
-<element name="FID-UL" library="SPCoast" package="FIDUCIAL_1MM" value="FID" x="6.35" y="92.075"/>
-<element name="FID-LR" library="SPCoast" package="FIDUCIAL_1MM" value="FID" x="93.98" y="7.62"/>
+<element name="U2X1" library="SPCoast" package="BOARD-10X8X2-TEMPLATE" value="BOARD" x="0" y="0"/>
+<element name="FID-UL" library="SPCoast" package="FIDUCIAL_1MM" value="FIDUCIAL" x="6.35" y="92.075"/>
+<element name="FID-LR" library="SPCoast" package="FIDUCIAL_1MM" value="FIDUCIAL" x="93.98" y="7.62"/>
 </elements>
 <signals>
