File: CMRI-Bus-Interface-L.brd (EAGLE design)
At the start: 50 x 80.5 mm, 23 parts, among them CON1 0.100, CON2 0.100, M1 MOUNTINGHOLE, M2 MOUNTINGHOLE, M3 MOUNTINGHOLE, M4 MOUNTINGHOLE, U1 MAX3465CSD, U2 NE555

Commit message: added values for connectors
Parts:
- J1: value (none) -> 0.100
Changed lines of the file:
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@@
 <setting verticaltext="up"/>
 </settings>
-<grid distance="50" unitdist="mil" unit="mil" style="dots" multiple="2" display="yes" altdistance="5" altunitdist="mil" altunit="mil"/>
+<grid distance="50" unitdist="mil" unit="mil" style="dots" multiple="2" display="yes" altdistance="25" altunitdist="mil" altunit="mil"/>
 <layers>
 <layer number="1" name="Top" color="4" fill="1" visible="yes" active="yes"/>
@@
 <attribute name="VALUE" x="41.402" y="17.78" size="1.27" layer="27" font="vector" rot="R90"/>
 </element>
-<element name="J1" library="SPCoast" package="J3-254" value="" x="36.195" y="38.1" smashed="yes" rot="R90">
+<element name="J1" library="SPCoast" package="J3-254" value="0.100" x="36.195" y="38.1" smashed="yes" rot="R90">
 <attribute name="NAME" x="41.704" y="36.704" size="1.27" layer="25" ratio="10" rot="R90"/>
 <attribute name="VALUE" x="39.703" y="34.164" size="1.27" layer="27" ratio="10" rot="R90"/>

Commit message: normalized values
Parts:
- C2, C4, C5: value .01uF -> 0.01uF
Changed lines of the file:
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@@
 <attribute name="VALUE" x="31.115" y="16.891" size="1.016" layer="21" font="vector" ratio="15" rot="R90"/>
 </element>
-<element name="C2" library="SPCoast" package="0603-CAP" value=".01uF" x="29.21" y="10.16" smashed="yes" rot="R270">
+<element name="C2" library="SPCoast" package="0603-CAP" value="0.01uF" x="29.21" y="10.16" smashed="yes" rot="R270">
 <attribute name="NAME" x="27.305" y="7.62" size="1.016" layer="25" font="vector" ratio="10" rot="R270"/>
 <attribute name="VALUE" x="27.051" y="12.446" size="1.016" layer="27" font="vector" ratio="10" rot="R270"/>
 </element>
-<element name="C4" library="SPCoast" package="0603-CAP" value=".01uF" x="13.716" y="14.224" smashed="yes">
+<element name="C4" library="SPCoast" package="0603-CAP" value="0.01uF" x="13.716" y="14.224" smashed="yes">
 <attribute name="NAME" x="9.906" y="13.589" size="1.016" layer="25" font="vector" ratio="10"/>
 <attribute name="VALUE" x="12.446" y="11.684" size="1.016" layer="27" font="vector" ratio="10"/>
 </element>
-<element name="C5" library="SPCoast" package="0603-CAP" value=".01uF" x="19.431" y="10.16" smashed="yes" rot="R270">
+<element name="C5" library="SPCoast" package="0603-CAP" value="0.01uF" x="19.431" y="10.16" smashed="yes" rot="R270">
 <attribute name="NAME" x="19.431" y="6.985" size="1.016" layer="25" font="vector" ratio="10" rot="R270"/>
 <attribute name="VALUE" x="17.526" y="12.7" size="1.016" layer="27" font="vector" ratio="10" rot="R270"/>
